Commit message: Add files via upload

File: Project 2/my_robot/urdf/my_robot.xacro (robot description, xacro)
@@ -22,5 +22,5 @@
       <origin xyz="0 0 0" rpy=" 0 0 0"/>
       <geometry>
-        <box size=".4 .2 .1"/>
+        <cylinder length="0.1" radius="0.2"/>
       </geometry>
     </collision>
@@ -28,5 +28,5 @@
       <origin xyz="0 0 0" rpy=" 0 0 0"/>
       <geometry>
-        <box size=".4 .2 .1"/>
+        <cylinder length="0.1" radius="0.2"/>
       </geometry>
     </visual>
@@ -70,5 +70,5 @@
       <origin  xyz="0 0 0" rpy="0 1.5707 1.5707"/>
       <geometry>
-        <cylinder length="0.05" radius="0.1"/>
+        <cylinder length="0.03" radius="0.1"/>
       </geometry>
     </collision>
@@ -76,5 +76,5 @@
       <origin xyz="0 0 0" rpy="0 1.5707 1.5707"/>
       <geometry>
-        <cylinder length="0.05" radius="0.1"/>
+        <cylinder length="0.03" radius="0.1"/>
       </geometry>
     </visual>
@@ -94,5 +94,5 @@
       <origin  xyz="0 0 0" rpy="0 1.5707 1.5707"/>
       <geometry>
-        <cylinder length="0.05" radius="0.1"/>
+        <cylinder length="0.03" radius="0.1"/>
       </geometry>
     </collision>
@@ -100,5 +100,5 @@
       <origin xyz="0 0 0" rpy="0 1.5707 1.5707"/>
       <geometry>
-        <cylinder length="0.05" radius="0.1"/>
+        <cylinder length="0.03" radius="0.1"/>
       </geometry>
     </visual>
@@ -135,13 +135,13 @@
     </inertial>
     <visual name='camera_visual'>
-      <origin xyz="0 0 0" rpy="0 0 0"/>
+      <origin xyz="0 0 0" rpy="1.5707 0 1.5707"/>
       <geometry>
-        <box size=".05 .05 .05"/>
+        <cylinder length="0.05" radius="0.025"/>
       </geometry>
     </visual>
     <collision name='camera_collision'>
-      <origin xyz="0 0 0" rpy="0 0 0"/>
+      <origin xyz="0 0 0" rpy="1.5707 0 1.5707"/>
       <geometry>
-        <box size=".05 .05 .05"/>
+        <cylinder length="0.05" radius="0.025"/>
       </geometry>
     </collision>
@@ -186,8 +186,8 @@
   </joint>
 <gazebo reference="left_wheel">
-    <material>Gazebo/Green</material>
+    <material>Gazebo/Yellow</material>
 </gazebo>
 <gazebo reference="right_wheel">
-    <material>Gazebo/Green</material>
+    <material>Gazebo/Yellow</material>
 </gazebo>
 <gazebo reference="camera">
@@ -195,5 +195,5 @@
 </gazebo>
 <gazebo reference="chassis">
-    <material>Gazebo/Blue</material>
+    <material>Gazebo/Green</material>
 </gazebo>
 </robot>
